File: Thermal_Camera/Thermal_Camera.kicad_sch (KiCad schematic)
At the start: 0 parts

Commit message: Schematic
Drew up Schematic
Parts:
- added A1: MLX90640ESF-BAA-000-TU, EasyEDA:TO-39_4P-BD9.3_MLX90640ESF-BAA-000-TU_H5.7, symbol MLX90640ESF-BAA-000-TU:MLX90640ESF-BAA-000-TU
- added C1, C3, C4, C5: 10uF, symbol Device:C_Small
- added C10, C11, C13, C14, C16, C19, C2, C8, C9: 0.1uF, symbol Device:C_Small
- added C12: 1uF, symbol Device:C_Small
- added C15, C17, C18: 4.7uF, symbol Device:C_Small
- added C6, C7: 22uF, symbol Device:C_Small
- added J1: USB_C_Receptacle_USB2.0, EasyEDA:USB-C_SMD-TYPE-C-31-M-12_1, symbol downloader-rescue:USB_C_Receptacle_USB2.0-Connector
- added J2: 5051101592, Thermal Camera Project:CON_5051101592_MOL, symbol 2026-03-02_00-05-03:5051101592
- added J3: 1040310811, EasyEDA:TF-SMD_TF-01A, symbol 2026-03-02_00-23-13:1040310811
- added J4: B2B-PH-K-S, EasyEDA:CONN-TH_B2B-PH-K-S, symbol B2B-PH-K-S:B2B-PH-K-S
- added L1: 2.2uH, symbol Device:L_Small
- added LED1: LTST-C170KGKT, EasyEDA:LED0603-RD, symbol 2026-03-02_00-25-59:LTST-C170KGKT
- added Q1: AO3400A, Package_TO_SOT_SMD:SOT-23, symbol Transistor_FET:AO3400A
- added R1, R2: 5.1k, symbol Device:R_Small
- added R10, R11, R13: 100k, symbol Device:R_Small
- added R12: 330, symbol Device:R_Small
- added R14: 100, symbol Device:R_Small
- added R15, R16, R17, R6, R7: 10k, symbol Device:R_Small
- added R3, R4: 22, symbol Device:R_Small
- added R5: 1.2k, symbol Device:R_Small_US
- added R8, R9: 4.7k, symbol Device:R_Small
- added SW1: PCM12SMTR, EasyEDA:SW-SMD_PCM12SMTR, symbol PCM12SMTR:PCM12SMTR
- added SW2, SW3, SW4: TS-1088R-02526, EasyEDA:SW-SMD_4P-L5.1-W5.1-P3.70-LS6.5-TL_H1.5, symbol Switch:SW_SPST
- added U1: TPB4056A20-ES1R, ESOP-8_TPK, symbol 2026-03-02_00-11-47:TPB4056A20-ES1R
- added U2: AP63203WU-7, EasyEDA:TSOT-26_L2.9-W1.6-P0.95-LS2.8-BL, symbol 2026-03-02_00-08-42:AP63203WU-7
- added U3: USBLC6-2SC6, EasyEDA:SOT-23-6_L2.9-W1.6-P0.95-LS2.8-BL, symbol Power_Protection:USBLC6-2SC6
- added U4: ESP32-S3-WROOM-1-N8R2, EasyEDA:WIRELM-SMD_ESP32-S3-WROOM-1, symbol ESP32-S3-WROOM-1-N8R2:ESP32-S3-WROOM-1-N8R2
Connections:
- new net: R12.1, U4.15 (IO3)
- new net: LED1.1, R12.2
- new net: R9.1, U4.17 (IO9)
- new net: C5.2, SW1.1, U2.2 (EN), U2.3 (VIN)
- new net: C8.2, L1.1, U2.5 (SW)
- new net: C8.1, U2.6 (BST)
- new net: Q1.1 (G), R13.2, R14.1
- new net: R4.2, U3.4 (I/O2)
- new net: R8.1, U4.12 (IO8)
- new net: R3.2, U3.6 (I/O1)
- new net: J1.A6 (D+), J1.B6 (D+), U3.1 (I/O1)
- new net: J1.A7 (D-), J1.B7 (D-), U3.3 (I/O2)
- new net: J2.14, J2.15, Q1.3 (D)
- new net: C13.2, R6.1, U4.3 (EN)
- new net: C3.1, U1.1 (VCC)
- new net: R5.1, U1.7 (IREF)
- new net: J1.A5 (CC1), R1.1
- new net: R7.1, U4.27 (IO0)
- new net: R10.1, R11.1, U4.7 (IO7)
- new net: J1.B5 (CC2), R2.1
- new net +3V3: A1.2 (VDD), C10.2, C11.2, C12.2, C14.2, C15.2, C16.1, C17.1, C18.1, C19.1, C6.1, C7.1, C9.2, J2.11, J2.13, J2.2, J2.3, J3.4 (VDD), L1.2, R6.2, U2.1 (FB), U4.2 (3V3)
- new net 3V3: R7.2
- new net BAT+: C4.1, J4.1, R11.2, SW1.2, U1.8 (BAT)
- new net GND: A1.3 (GND), C1.1, C1.2, C10.1, C11.1, C12.1, C13.1, C14.1, C15.1, C16.2, C17.2, C18.2, C19.2, C2.1, C2.2, C3.2, C4.2, C5.1, C6.2, C7.2, C9.1, J1.A1 (GND), J1.A12 (GND), J1.A4 (VBUS), J1.A9 (VBUS), J1.B1 (GND), J1.B12 (GND), J1.B4 (VBUS), J1.B9 (VBUS), J1.S1 (SHIELD), J2.1, J2.10, J2.7, J3.6 (VSS), J4.2, LED1.2, Q1.2 (S), R1.2, R10.2, R13.1, R15.2, R16.2, R17.2, R2.2, R5.2, SW1.S1 (SHIELD), SW1.S2 (SHIELD__1), SW1.S3 (SHIELD__2), SW1.S4 (SHIELD__3), SW2.2 (B), SW3.2 (B), SW4.2 (B), U1.4 (EN), U1.5 (GND), U1.6 (IMIN), U1.9 (GND), U2.4 (GND), U3.2 (GND), U3.5 (VBUS), U4.1 (GND), U4.40 (GND__1), U4.41_1 (GND__2), U4.41_2 (GND__3), U4.41_3 (GND__4), U4.41_4 (GND__5), U4.41_5 (GND__6), U4.41_6 (GND__7), U4.41_7 (GND__8), U4.41_8 (GND__9), U4.41_9 (GND__10)
- new net GWM: R14.2, U4.34 (IO41)
- new net I2C_SCL: A1.4 (SCL), R9.2
- new net I2C_SDA: A1.1 (SDA), R8.2
- new net SD_CS: J3.2 (CD/DAT3), U4.32 (IO39)
- new net SPI_MISO: J3.7 (DAT0), U4.30 (IO37)
- new net SPI_MOSI: J2.6, J3.3 (CMD), U4.28 (IO35)
- new net SPI_SCK: J2.9, J3.5 (CLK), U4.29 (IO36)
- new net SW_DOWN: R16.1, SW3.1 (A), U4.5 (IO5)
- new net SW_MENU: R17.1, SW4.1 (A), U4.6 (IO6)
- new net SW_UP: R15.1, SW2.1 (A), U4.4 (IO4)
- new net TFT_CS: J2.4, U4.23 (IO21)
- new net TFT_DC: J2.8, U4.31 (IO38)
- new net TFT_RST: J2.5, U4.33 (IO40)
- new net USB_D+: R3.1, U4.14 (IO20)
- new net USB_D-: R4.1, U4.13 (IO19)
- no-connect marks 0 -> 10
Other:
- note added: "3V3 BUCK REGULATOR"
- note added: "Battery Connector"
- note added: "CHARGER"
- note added: "DISPLAY + SD"
- note added: "ESP32 3V3 CAPS"
- note added: "ESP32 S3"
- note added: "MLX90640"
- note added: "Power ON/OFF"
- note added: "SD-CARD"
- note added: "SWITCHES"
- note added: "USB-C"

Commit message: New Libraries
Modified component choice, added new capacitor, and created new libraries
Parts:
- added C20: 10uF, symbol Device:C_Small
- C13: value 0.1uF -> 1uF
- L1: value 2.2uH -> 3.9uH
Connections:
- net +3V3: now also C20.2
- net GND: now also C20.1
Other:
- moved on the sheet: C13
Changed lines of the file:
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@@
 	)
 	(junction
+		(at 293.37 137.16)
+		(diameter 0)
+		(color 0 0 0 0)
+	)
+	(junction
 		(at 31.75 115.57)
 		(diameter 0)
@@
 	(wire
 		(pts
+			(xy 293.37 137.16) (xy 300.99 137.16)
+		)
+		(stroke
+			(width 0)
+			(type default)
+		)
+	)
+	(wire
+		(pts
 			(xy 52.07 46.99) (xy 64.77 46.99)
 		)
@@
 	)
 	(symbol
+		(lib_id "Device:C_Small")
+		(at 300.99 139.7 180)
+		(unit 1)
+		(exclude_from_sim no)
+		(in_bom yes)
+		(on_board yes)
+		(dnp no)
+		(property "Reference" "C20"
+			(at 295.402 139.7 0)
+			(effects
+				(font
+					(size 1.27 1.27)
+				)
+				(justify right)
+			)
+		)
+		(property "Value" "10uF"
+			(at 295.148 141.224 0)
+			(effects
+				(font
+					(size 1.27 1.27)
+				)
+				(justify right)
+				(hide yes)
+			)
+		)
+		(property "Footprint" ""
+			(at 300.99 139.7 0)
+			(effects
+				(font
+					(size 1.27 1.27)
+				)
+				(hide yes)
+			)
+		)
+		(property "Datasheet" "~"
+			(at 300.99 139.7 0)
+			(effects
+				(font
+					(size 1.27 1.27)
+				)
+				(hide yes)
+			)
+		)
+		(property "Description" "Unpolarized capacitor, small symbol"
+			(at 300.99 139.7 0)
+			(effects
+				(font
+					(size 1.27 1.27)
+				)
+				(hide yes)
+			)
+		)
+		(pin "1"
+		)
+		(pin "2"
+		)
+		(instances
+			(project "Thermal_Camera"
+				(path "/69bb2319-c70b-40cf-9602-3016c4fa9ddb"
+					(reference "C20")
+					(unit 1)
+				)
+			)
+		)
+	)
+	(symbol
 		(lib_id "Switch:SW_SPST")
 		(at 48.26 133.35 0)
@@
 	(symbol
 		(lib_id "power:GND")
+		(at 300.99 142.24 0)
+		(unit 1)
+		(exclude_from_sim no)
+		(in_bom yes)
+		(on_board yes)
+		(dnp no)
+		(fields_autoplaced yes)
+		(property "Reference" "#PWR053"
+			(at 300.99 148.59 0)
+			(effects
+				(font
+					(size 1.27 1.27)
+				)
+				(hide yes)
+			)
+		)
+		(property "Value" "GND"
+			(at 300.99 147.32 0)
+			(effects
+				(font
+					(size 1.27 1.27)
+				)
+			)
+		)
+		(property "Footprint" ""
+			(at 300.99 142.24 0)
+			(effects
+				(font
+					(size 1.27 1.27)
+				)
+				(hide yes)
+			)
+		)
+		(property "Datasheet" ""
+			(at 300.99 142.24 0)
+			(effects
+				(font
+					(size 1.27 1.27)
+				)
+				(hide yes)
+			)
+		)
+		(property "Description" "Power symbol creates a global label with name \"GND\" , ground"
+			(at 300.99 142.24 0)
+			(effects
+				(font
+					(size 1.27 1.27)
+				)
+				(hide yes)
+			)
+		)
+		(pin "1"
+		)
+		(instances
+			(project "Thermal_Camera"
+				(path "/69bb2319-c70b-40cf-9602-3016c4fa9ddb"
+					(reference "#PWR053")
+					(unit 1)
+				)
+			)
+		)
+	)
+	(symbol
+		(lib_id "power:GND")
 		(at 254 76.2 180)
 		(unit 1)
@@
 			)
 		)
-		(property "Value" "2.2uH"
+		(property "Value" "3.9uH"
 			(at 226.06 43.18 90)
 			(effects
@@
 	(symbol
 		(lib_id "Device:C_Small")
-		(at 262.89 44.45 180)
+		(at 262.89 44.45 0)
+		(mirror x)
 		(unit 1)
 		(exclude_from_sim no)
@@
 		(dnp no)
 		(property "Reference" "C13"
-			(at 256.54 44.45 0)
+			(at 269.24 44.45 0)
 			(effects
 				(font
@@
 			)
 		)
-		(property "Value" "0.1uF"
-			(at 255.016 45.466 0)
+		(property "Value" "1uF"
+			(at 270.764 45.466 0)
 			(effects
 				(font

Commit message: Component addition, Schematic revision, and Layout
Added LED booster driver IC for LCD screen, updated libraries, and got the general layout finished, I need to calculate screen and battery dimensions for the final revisions.
Parts:
- removed Q1: AO3400A, Package_TO_SOT_SMD:SOT-23, symbol Transistor_FET:AO3400A
- removed R14: 100, symbol Device:R_Small
- added C21, C22: 1uF, Capacitor_SMD:C_0805_2012Metric_Pad1.18x1.45mm_HandSolder, symbol Device:C_Small
- added D1: D_Schottky, Thermal Footprints:SOD2512X115N, symbol Device:D_Schottky
- added L2: 3.9uH, Thermal Footprints:IND_LQH2MCN4R7M02L, symbol Device:L_Small
- added U5: MP3302DJ-LF-Z, Thermal Footprints:SOT95P280X100-5N, symbol MP3302DJ-LF-Z:MP3302DJ-LF-Z
- A1: footprint EasyEDA:TO-39_4P-BD9.3_MLX90640ESF-BAA-000-TU_H5.7 -> Thermal Footprints:TO-39_4P-BD9.3_MLX90640ESF-BAA-000-TU_H5.7
- C1, C10, C11, C12, C13, C14, C15, C16, C17, C18, C19, C2, C20, C3, C4, C5, C6, C7, C8, C9: footprint (none) -> Capacitor_SMD:C_0805_2012Metric_Pad1.18x1.45mm_HandSolder
- J1: footprint EasyEDA:USB-C_SMD-TYPE-C-31-M-12_1 -> Connector_USB:USB_C_Receptacle_HRO_TYPE-C-31-M-12; symbol downloader-rescue:USB_C_Receptacle_USB2.0-Connector -> Connector:USB_C_Receptacle_USB2.0_16P
- J2: footprint Thermal Camera Project:CON_5051101592_MOL -> Thermal Footprints:CON_5051101592_MOL
- J3: footprint EasyEDA:TF-SMD_TF-01A -> Thermal Footprints:104031-0811_MOL
- J4: footprint EasyEDA:CONN-TH_B2B-PH-K-S -> Thermal Footprints:CONN-TH_B2B-PH-K-S
- L1: footprint (none) -> Thermal Footprints:IND_4030
- LED1: footprint EasyEDA:LED0603-RD -> Thermal Footprints:LED0603-RD
- R1, R10, R11, R12, R15, R16, R17, R2, R3, R4, R6, R7, R8, R9: footprint (none) -> Resistor_SMD:R_0805_2012Metric_Pad1.20x1.40mm_HandSolder
- R13: value 100k -> 5; footprint (none) -> Resistor_SMD:R_0805_2012Metric_Pad1.20x1.40mm_HandSolder
- R5: footprint (none) -> Resistor_SMD:R_0805_2012Metric_Pad1.20x1.40mm_HandSolder; symbol Device:R_Small_US -> Device:R
- SW1: footprint EasyEDA:SW-SMD_PCM12SMTR -> Thermal Footprints:SW-SMD_PCM12SMTR
- SW2, SW3, SW4: footprint EasyEDA:SW-SMD_4P-L5.1-W5.1-P3.70-LS6.5-TL_H1.5 -> Thermal Footprints:SW-SMD_4P-L5.1-W5.1-P3.70-LS6.5-TL_H1.5
- U1: footprint ESOP-8_TPK -> Thermal Footprints:ESOP-8_L4.9-W3.9-P1.27-LS6.0-BL-EP
- U2: footprint EasyEDA:TSOT-26_L2.9-W1.6-P0.95-LS2.8-BL -> Thermal Footprints:TSOT-26_L2.9-W1.6-P0.95-LS2.8-BL
- U3: footprint EasyEDA:SOT-23-6_L2.9-W1.6-P0.95-LS2.8-BL -> Thermal Footprints:SOT-23-6
- U4: footprint EasyEDA:WIRELM-SMD_ESP32-S3-WROOM-1 -> Thermal Footprints:WIRELM-SMD_ESP32-S3-WROOM-1
Connections:
- net 3V3 is gone; now on net +3V3: R7.2
- net +3V3: now also C21.1, U5.5 (IN); no longer J2.13
- net BAT+: now also R11.1; no longer R11.2
- net GND: now also J1.SH (SHIELD), J2.14, J2.15, J2.S1, J2.S2, R13.2, C21.2, C22.2, U5.2 (GND); no longer C1.1, C2.1, J1.A4 (VBUS), J1.A9 (VBUS), J1.B4 (VBUS), J1.B9 (VBUS), J1.S1 (SHIELD), R13.1, U1.4 (EN), U3.5 (VBUS)
- net GWM: now also U5.4 (EN)
- net VBUS_5V: now reaches C3.1, U1.1 (VCC)
- net VBUS_5V: now also C1.1, C2.1, J1.A4 (VBUS), J1.A9 (VBUS), J1.B4 (VBUS), J1.B9 (VBUS), U1.4 (EN), U3.5 (VBUS)
- net at R10.1, U4.7 (IO7): now also R11.2; no longer R11.1
- new net: L2.1, U5.1 (SW)
- new net: R13.1, U5.3 (FB)
- new net: C22.1, D1.C (K), J2.13
- new net: D1.A, L2.2
- no-connect marks 10 -> 28
Other:
- note added: "BATTERY CHARGER"
- note added: "DISPLAY + LED DRIVER + SD"
- note added: "THERMAL SENSOR"
- note removed: "CHARGER"
- note removed: "DISPLAY + SD"
- note removed: "MLX90640"
- moved on the sheet: A1, C1, C14, C15, C16, C17, C2, C4, C5, J2, R11, R15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
